Commit message: 脚底碰撞改为 7 个圆柱近似（URDF + MJCF）
ankle_roll_l_link / ankle_roll_r_link 的碰撞体由整块脚底网格改为
7 个圆柱，参数取自参考资产包的脚底设计。

URDF（3 份）：urdf/tiangong3.urdf、tiangong3_brainco.urdf、tiangong3_inspire.urdf
- ankle_roll_{l,r}_link：1 个 mesh collision -> 7 个命名 cylinder collision

MJCF（2 份）：mujoco/tiangong3_torq.xml、tiangong3_simplify.xml
- ankle_roll_{l,r}_link：1 个 mesh collision geom -> 7 个 cylinder geom
- 保留 class="collision"，继承 condim/contype/conaffinity/solref/solimp/friction

未改动：所有 STL、inertial、joint、visual、其他 link 的碰撞，以及 MJCF 的
default(13)、exclude(38)、sensor(5)、option。

已知影响：7 个圆柱最低点 -0.058 m，比原脚底网格最低点 -0.056774 m 低
1.23 mm；两份 MJCF 的 floor 高度仍按原网格自动计算，默认姿态下脚底存在
约 1.23 mm（torq）/ 0.6 mm（simplify）的初始穿透。

README 已补充「脚底碰撞体」与「脚底碰撞」两节说明。

验证：3 份 URDF 与参考包逐字段一致；2 份 MJCF 的 7 组 cylinder 参数
逐字段一致；MuJoCo 3.10.0 编译通过（nbody=40, ngeom=91, cylinder_geom=14）。

File: urdf/tiangong3.urdf (robot description, URDF)
Before this commit: robot tiangong3_urdf, 39 links, 38 joints
Links:
- link ankle_roll_l_link: geometry collision cylinder length=0.06 radius=0.012; collision cylinder length=0.06 radius=0.012
- link ankle_roll_r_link: geometry collision cylinder length=0.06 radius=0.012; collision cylinder length=0.06 radius=0.012

File: urdf/tiangong3_brainco.urdf (robot description, URDF)
Before this commit: robot tiangong3_brainco, 83 links, 82 joints
Links:
- link ankle_roll_l_link: geometry collision cylinder length=0.06 radius=0.012; collision cylinder length=0.06 radius=0.012
- link ankle_roll_r_link: geometry collision cylinder length=0.06 radius=0.012; collision cylinder length=0.06 radius=0.012

File: urdf/tiangong3_inspire.urdf (robot description, URDF)
Before this commit: robot tiangong3_inspire, 101 links, 100 joints
Links:
- link ankle_roll_l_link: geometry collision cylinder length=0.06 radius=0.012; collision cylinder length=0.06 radius=0.012
- link ankle_roll_r_link: geometry collision cylinder length=0.06 radius=0.012; collision cylinder length=0.06 radius=0.012
